File: _autosave-TLI5012B.sch (KiCad schematic (older format))
At the start: 4 parts, among them J1 Conn_01x05_Female, U1 TLI5012B

Commit message: with mounting holes
Parts:
- U1: footprint Package_SO:SO-8_5.3x6.2mm_P1.27mm -> Package_SO:SOP-8_3.76x4.96mm_P1.27mm
Changed lines of the file:
@@
 F 0 "U1" H 5400 3865 50  0000 C CNN
 F 1 "TLI5012B" H 5400 3774 50  0000 C CNN
-F 2 "Package_SO:SO-8_5.3x6.2mm_P1.27mm" H 5500 3250 50  0001 C CNN
+F 2 "Package_SO:SOP-8_3.76x4.96mm_P1.27mm" H 5500 3250 50  0001 C CNN
 F 3 "" H 5500 3250 50  0001 C CNN
 	1    5400 3450
