File: TLI5012B.sch (KiCad schematic (older format))
At the start: 2 parts, among them J1 Conn_01x08_Female, U1 TLI5012B

Commit message: with jst connector
Parts:
- removed J1: Conn_01x08_Female, Connector_PinHeader_2.54mm:PinHeader_1x08_P2.54mm_Vertical, symbol Connector:Conn_01x08_Female
- added D1: LED, LED_SMD:LED_0603_1608Metric, symbol Device:LED
- added J1: Conn_01x05_Female, Connector_JST:JST_SH_SM05B-SRSS-TB_1x05-1MP_P1.00mm_Horizontal, symbol Connector:Conn_01x05_Female
- added R1: 1k, LED_SMD:LED_0402_1005Metric, symbol Device:R
- U1: symbol custom:TLI5012B -> TLI5012B-rescue:TLI5012B-custom
Connections:
- net GND: now also D1.1 (K), J1.4 (Pin_4)
- net IFA: now also J1.2 (Pin_2), R1.1
- net IFB: now also J1.1 (Pin_1)
- net IFC: now also J1.3 (Pin_3)
- net VDD: now also J1.5 (Pin_5)
- new net: D1.2 (A), R1.2
Changed lines of the file:
@@
 EESchema Schematic File Version 4
 LIBS:TLI5012B-cache
-EELAYER 30 0
+EELAYER 29 0
 EELAYER END
 $Descr A4 11693 8268
@@
 $EndDescr
 $Comp
-L custom:TLI5012B U1
+L TLI5012B-rescue:TLI5012B-custom U1
 U 1 1 5D38797F
 P 5400 3450
@@
 F 3 "" H 5500 3250 50  0001 C CNN
 	1    5400 3450
-	1    0    0    -1
-$EndComp
-$Comp
-L Connector:Conn_01x08_Female J1
-U 1 1 5D387A4C
-P 6700 3350
-F 0 "J1" V 6865 3280 50  0000 C CNN
-F 1 "Conn_01x08_Female" V 6774 3280 50  0000 C CNN
-F 2 "Connector_PinHeader_2.54mm:PinHeader_1x08_P2.54mm_Vertical" H 6700 3350 50  0001 C CNN
-F 3 "~" H 6700 3350 50  0001 C CNN
-	1    6700 3350
 	1    0    0    -1
 $EndComp
@@
 Text Label 5000 3600 2    50   ~ 0
 DATA
-Text Label 6500 3150 2    50   ~ 0
+$Comp
+L Connector:Conn_01x05_Female J1
+U 1 1 5D397F17
+P 6800 3400
+F 0 "J1" H 6828 3426 50  0000 L CNN
+F 1 "Conn_01x05_Female" H 6828 3335 50  0000 L CNN
+F 2 "Connector_JST:JST_SH_SM05B-SRSS-TB_1x05-1MP_P1.00mm_Horizontal" H 6800 3400 50  0001 C CNN
+F 3 "~" H 6800 3400 50  0001 C CNN
+	1    6800 3400
+	1    0    0    -1
+$EndComp
+Text Label 6600 3200 2    50   ~ 0
+IFB
+Text Label 6600 3300 2    50   ~ 0
+IFA
+Text Label 6600 3400 2    50   ~ 0
+IFC
+Text Label 6600 3500 2    50   ~ 0
+GND
+Text Label 6600 3600 2    50   ~ 0
 VDD
-Text Label 6500 3050 2    50   ~ 0
+$Comp
+L Device:LED D1
+U 1 1 5D397E81
+P 6150 4500
+F 0 "D1" V 6189 4383 50  0000 R CNN
+F 1 "LED" V 6098 4383 50  0000 R CNN
+F 2 "LED_SMD:LED_0603_1608Metric" H 6150 4500 50  0001 C CNN
+F 3 "~" H 6150 4500 50  0001 C CNN
+	1    6150 4500
+	0    -1   -1   0
+$EndComp
+$Comp
+L Device:R R1
+U 1 1 5D398A35
+P 6150 4200
+F 0 "R1" H 6220 4246 50  0000 L CNN
+F 1 "1k" H 6220 4155 50  0000 L CNN
+F 2 "LED_SMD:LED_0402_1005Metric" V 6080 4200 50  0001 C CNN
+F 3 "~" H 6150 4200 50  0001 C CNN
+	1    6150 4200
+	1    0    0    -1
+$EndComp
+Text Label 6150 4650 3    50   ~ 0
 GND
-Text Label 6500 3250 2    50   ~ 0
+Text Label 6150 4050 1    50   ~ 0
 IFA
-Text Label 6500 3350 2    50   ~ 0
-IFB
-Text Label 6500 3450 2    50   ~ 0
-IFC
-Text Label 6500 3650 2    50   ~ 0
-CSQ
-Text Label 6500 3750 2    50   ~ 0
-SCK
-Text Label 6500 3550 2    50   ~ 0
-DATA
 $EndSCHEMATC

Commit message: with mounting holes
Parts:
- U1: footprint Package_SO:SO-8_5.3x6.2mm_P1.27mm -> Package_SO:SOIC-8_5.23x5.23mm_P1.27mm
Changed lines of the file:
@@
 F 0 "U1" H 5400 3865 50  0000 C CNN
 F 1 "TLI5012B" H 5400 3774 50  0000 C CNN
-F 2 "Package_SO:SO-8_5.3x6.2mm_P1.27mm" H 5500 3250 50  0001 C CNN
+F 2 "Package_SO:SOIC-8_5.23x5.23mm_P1.27mm" H 5500 3250 50  0001 C CNN
 F 3 "" H 5500 3250 50  0001 C CNN
 	1    5400 3450

Commit message: with mounting holes
Parts:
- U1: footprint Package_SO:SOIC-8_5.23x5.23mm_P1.27mm -> Package_SO:SOP-8_3.76x4.96mm_P1.27mm
Changed lines of the file:
@@
 F 0 "U1" H 5400 3865 50  0000 C CNN
 F 1 "TLI5012B" H 5400 3774 50  0000 C CNN
-F 2 "Package_SO:SOIC-8_5.23x5.23mm_P1.27mm" H 5500 3250 50  0001 C CNN
+F 2 "Package_SO:SOP-8_3.76x4.96mm_P1.27mm" H 5500 3250 50  0001 C CNN
 F 3 "" H 5500 3250 50  0001 C CNN
 	1    5400 3450
