File: TLI5012B/TLI5012B.sch (KiCad schematic (older format))
At the start: 4 parts, among them J1 Conn_01x05_Female, U1 TLI5012B

Commit message: with pcb for walkera_wk-ws-028-014A
Parts:
- removed D1: LED, LED_SMD:LED_0603_1608Metric, symbol Device:LED
- removed R1: 1k, LED_SMD:LED_0402_1005Metric, symbol Device:R
- added C1: C, Capacitor_SMD:C_0402_1005Metric, symbol Device:C
- added H1, H2, H3, H4: MountingHole, MountingHole:MountingHole_3.2mm_M3, symbol Mechanical:MountingHole
- J1: footprint Connector_JST:JST_SH_SM05B-SRSS-TB_1x05-1MP_P1.00mm_Horizontal -> Connector_PinHeader_2.54mm:PinHeader_1x05_P2.54mm_Vertical
- U1: footprint Package_SO:SO-8_5.3x6.2mm_P1.27mm -> custom_lib:TLI5012B
Connections:
- net GND: now also C1.2
- net IFA: now also J1.3 (Pin_3); no longer J1.2 (Pin_2)
- net IFB: now also J1.2 (Pin_2); no longer J1.1 (Pin_1)
- net IFC: now also J1.1 (Pin_1); no longer J1.3 (Pin_3)
- net VDD renamed +5V
- net +5V: now also C1.1
Other:
- moved on the sheet: J1
Changed lines of the file:
@@
 EESchema Schematic File Version 4
 LIBS:TLI5012B-cache
-EELAYER 29 0
+EELAYER 26 0
 EELAYER END
 $Descr A4 11693 8268
@@
 F 0 "U1" H 5400 3865 50  0000 C CNN
 F 1 "TLI5012B" H 5400 3774 50  0000 C CNN
-F 2 "Package_SO:SO-8_5.3x6.2mm_P1.27mm" H 5500 3250 50  0001 C CNN
+F 2 "custom_lib:TLI5012B" H 5500 3250 50  0001 C CNN
 F 3 "" H 5500 3250 50  0001 C CNN
 	1    5400 3450
@@
 Text Label 5800 3300 0    50   ~ 0
 IFB
-Text Label 5800 3400 0    50   ~ 0
-GND
-Text Label 5800 3500 0    50   ~ 0
-VDD
 Text Label 5800 3600 0    50   ~ 0
 IFA
@@
 L Connector:Conn_01x05_Female J1
 U 1 1 5D397F17
-P 6800 3400
-F 0 "J1" H 6828 3426 50  0000 L CNN
-F 1 "Conn_01x05_Female" H 6828 3335 50  0000 L CNN
-F 2 "Connector_JST:JST_SH_SM05B-SRSS-TB_1x05-1MP_P1.00mm_Horizontal" H 6800 3400 50  0001 C CNN
-F 3 "~" H 6800 3400 50  0001 C CNN
-	1    6800 3400
+P 6875 3450
+F 0 "J1" H 6903 3476 50  0000 L CNN
+F 1 "Conn_01x05_Female" H 6903 3385 50  0000 L CNN
+F 2 "Connector_PinHeader_2.54mm:PinHeader_1x05_P2.54mm_Vertical" H 6875 3450 50  0001 C CNN
+F 3 "~" H 6875 3450 50  0001 C CNN
+	1    6875 3450
 	1    0    0    -1
 $EndComp
-Text Label 6600 3200 2    50   ~ 0
+Text Label 6675 3350 2    50   ~ 0
 IFB
-Text Label 6600 3300 2    50   ~ 0
+Text Label 6675 3450 2    50   ~ 0
 IFA
-Text Label 6600 3400 2    50   ~ 0
+Text Label 6675 3250 2    50   ~ 0
 IFC
-Text Label 6600 3500 2    50   ~ 0
-GND
-Text Label 6600 3600 2    50   ~ 0
-VDD
 $Comp
-L Device:LED D1
-U 1 1 5D397E81
-P 6150 4500
-F 0 "D1" V 6189 4383 50  0000 R CNN
-F 1 "LED" V 6098 4383 50  0000 R CNN
-F 2 "LED_SMD:LED_0603_1608Metric" H 6150 4500 50  0001 C CNN
-F 3 "~" H 6150 4500 50  0001 C CNN
-	1    6150 4500
+L Device:C C1
+U 1 1 5F7EEAC9
+P 6500 2775
+F 0 "C1" H 6615 2821 50  0000 L CNN
+F 1 "C" H 6615 2730 50  0000 L CNN
+F 2 "Capacitor_SMD:C_0402_1005Metric" H 6538 2625 50  0001 C CNN
+F 3 "~" H 6500 2775 50  0001 C CNN
+	1    6500 2775
+	1    0    0    -1
+$EndComp
+$Comp
+L power:+5V #PWR0101
+U 1 1 5F7EEB26
+P 6675 3650
+F 0 "#PWR0101" H 6675 3500 50  0001 C CNN
+F 1 "+5V" V 6690 3778 50  0000 L CNN
+F 2 "" H 6675 3650 50  0001 C CNN
+F 3 "" H 6675 3650 50  0001 C CNN
+	1    6675 3650
 	0    -1   -1   0
 $EndComp
 $Comp
-L Device:R R1
-U 1 1 5D398A35
-P 6150 4200
-F 0 "R1" H 6220 4246 50  0000 L CNN
-F 1 "1k" H 6220 4155 50  0000 L CNN
-F 2 "LED_SMD:LED_0402_1005Metric" V 6080 4200 50  0001 C CNN
-F 3 "~" H 6150 4200 50  0001 C CNN
-	1    6150 4200
+L power:+5V #PWR0102
+U 1 1 5F7EEB47
+P 5800 3500
+F 0 "#PWR0102" H 5800 3350 50  0001 C CNN
+F 1 "+5V" V 5815 3628 50  0000 L CNN
+F 2 "" H 5800 3500 50  0001 C CNN
+F 3 "" H 5800 3500 50  0001 C CNN
+	1    5800 3500
+	0    1    1    0
+$EndComp
+$Comp
+L power:GND #PWR0103
+U 1 1 5F7EEBB6
+P 6675 3550
+F 0 "#PWR0103" H 6675 3300 50  0001 C CNN
+F 1 "GND" V 6680 3422 50  0000 R CNN
+F 2 "" H 6675 3550 50  0001 C CNN
+F 3 "" H 6675 3550 50  0001 C CNN
+	1    6675 3550
+	0    1    1    0
+$EndComp
+$Comp
+L power:GND #PWR0104
+U 1 1 5F7EEBD1
+P 5800 3400
+F 0 "#PWR0104" H 5800 3150 50  0001 C CNN
+F 1 "GND" V 5805 3272 50  0000 R CNN
+F 2 "" H 5800 3400 50  0001 C CNN
+F 3 "" H 5800 3400 50  0001 C CNN
+	1    5800 3400
+	0    -1   -1   0
+$EndComp
+$Comp
+L power:GND #PWR0105
+U 1 1 5F7EEBE8
+P 6500 2925
+F 0 "#PWR0105" H 6500 2675 50  0001 C CNN
+F 1 "GND" V 6505 2797 50  0000 R CNN
+F 2 "" H 6500 2925 50  0001 C CNN
+F 3 "" H 6500 2925 50  0001 C CNN
+	1    6500 2925
+	0    -1   -1   0
+$EndComp
+$Comp
+L power:+5V #PWR0106
+U 1 1 5F7EEBF9
+P 6500 2625
+F 0 "#PWR0106" H 6500 2475 50  0001 C CNN
+F 1 "+5V" V 6515 2753 50  0000 L CNN
+F 2 "" H 6500 2625 50  0001 C CNN
+F 3 "" H 6500 2625 50  0001 C CNN
+	1    6500 2625
+	0    1    1    0
+$EndComp
+$Comp
+L Mechanical:MountingHole H1
+U 1 1 5F7EEEED
+P 7850 2725
+F 0 "H1" H 7950 2771 50  0000 L CNN
+F 1 "MountingHole" H 7950 2680 50  0000 L CNN
+F 2 "MountingHole:MountingHole_3.2mm_M3" H 7850 2725 50  0001 C CNN
+F 3 "~" H 7850 2725 50  0001 C CNN
+	1    7850 2725
 	1    0    0    -1
 $EndComp
-Text Label 6150 4650 3    50   ~ 0
-GND
-Text Label 6150 4050 1    50   ~ 0
-IFA
+$Comp
+L Mechanical:MountingHole H2
+U 1 1 5F7EEF1D
+P 7850 2900
+F 0 "H2" H 7950 2946 50  0000 L CNN
+F 1 "MountingHole" H 7950 2855 50  0000 L CNN
+F 2 "MountingHole:MountingHole_3.2mm_M3" H 7850 2900 50  0001 C CNN
+F 3 "~" H 7850 2900 50  0001 C CNN
+	1    7850 2900
+	1    0    0    -1
+$EndComp
+$Comp
+L Mechanical:MountingHole H3
+U 1 1 5F7EEF41
+P 7850 3075
+F 0 "H3" H 7950 3121 50  0000 L CNN
+F 1 "MountingHole" H 7950 3030 50  0000 L CNN
+F 2 "MountingHole:MountingHole_3.2mm_M3" H 7850 3075 50  0001 C CNN
+F 3 "~" H 7850 3075 50  0001 C CNN
+	1    7850 3075
+	1    0    0    -1
+$EndComp
+$Comp
+L Mechanical:MountingHole H4
+U 1 1 5F7EEF71
+P 7850 3250
+F 0 "H4" H 7950 3296 50  0000 L CNN
+F 1 "MountingHole" H 7950 3205 50  0000 L CNN
+F 2 "MountingHole:MountingHole_3.2mm_M3" H 7850 3250 50  0001 C CNN
+F 3 "~" H 7850 3250 50  0001 C CNN
+	1    7850 3250
+	1    0    0    -1
+$EndComp
 $EndSCHEMATC

Commit message: with 1.27 pitch
Parts:
- J1: footprint Connector_PinHeader_2.54mm:PinHeader_1x05_P2.54mm_Vertical -> Connector_PinHeader_1.27mm:PinHeader_1x05_P1.27mm_Vertical
Changed lines of the file:
@@
 F 0 "J1" H 6903 3476 50  0000 L CNN
 F 1 "Conn_01x05_Female" H 6903 3385 50  0000 L CNN
-F 2 "Connector_PinHeader_2.54mm:PinHeader_1x05_P2.54mm_Vertical" H 6875 3450 50  0001 C CNN
+F 2 "Connector_PinHeader_1.27mm:PinHeader_1x05_P1.27mm_Vertical" H 6875 3450 50  0001 C CNN
 F 3 "~" H 6875 3450 50  0001 C CNN
 	1    6875 3450
